File: gb_rom_board.kicad_pcb (KiCad board)
At the start: 2 copper layers, 51 x 60.6 mm, 3 parts, among them J1 PLCC, J2 DEV, J3 CART

Commit message: henkou
Parts:
- added G***: LOGO, doragasu-footprints:LOGO_GB, B.Cu at (138.4, 109.5)
- added G***: LOGO, doragasu-footprints:moji, B.Cu at (138.4, 91.2)
- added G***: LOGO, doragasu-footprints:mizunomi, F.Cu at (138.4, 108.0)
